Commit message: fixed urdf for gazebo

File: ceres_description/urdf/ceres.urdf.xacro (robot description, xacro)
@@ -20,6 +20,6 @@
   <xacro:property name="wheel_radius" value="0.135"/>
   <xacro:property name="axis_height" value="-0.03"/>
-  <xacro:property name="axis_left" value="${-body_width/2 - wheel_body_offset}"/>
-  <xacro:property name="axis_right" value="${body_width/2 + wheel_body_offset}"/>
+  <xacro:property name="axis_right" value="${-body_width/2 - wheel_body_offset}"/>
+  <xacro:property name="axis_left" value="${body_width/2 + wheel_body_offset}"/>
   <xacro:property name="axis_length" value="${body_width + 2 * wheel_body_offset}" />
   <xacro:property name="turning_adaptation" value="0.95" />
@@ -45,5 +45,4 @@
       <origin xyz="0 0 0" rpy="0 0 0" />
       <geometry>
-        <!--mesh filename="package://pluto_description/meshes/pluto_base.stl"/-->
         <box size="${body_length} ${body_width} ${body_height}"/>
       </geometry>
@@ -56,5 +55,4 @@
       <geometry>
         <box size="${body_length} ${body_width} ${body_height}"/>
-        <!--mesh filename="package://pluto_description/meshes/pluto_base_collision.stl"/-->
       </geometry>
     </collision>
@@ -66,5 +64,4 @@
   </link>
   <joint name="base_footprint_to_base_joint" type="fixed">
-    <!-- origin xyz="0 0 0.2" rpy="0 ${-M_PI/18.0} 0" /-->
     <origin xyz="0 0 ${wheel_radius - axis_height}" rpy="0 0 0" />
     <parent link="base_footprint"/>
@@ -77,6 +74,5 @@
         <origin xyz="0 0 0" rpy="${M_PI/2} 0 0" />
         <geometry>
-          <!--mesh filename="package://pluto_description/meshes/pluto_wheel.stl"/-->
-	  <cylinder length="${wheel_thickness}" radius="${wheel_radius}"/>
+          <cylinder length="${wheel_thickness}" radius="${wheel_radius}"/>
         </geometry>
         <material name="black" >
@@ -85,8 +81,7 @@
       </visual>
       <collision>
-        <origin xyz="0 0 0" rpy="0 0 0" />
-        <geometry>
-	  <cylinder length="${wheel_thickness}" radius="${wheel_radius}"/>
-          <!-- mesh filename="package://pluto_description/meshes/pluto_wheel_collision.stl"/-->
+        <origin xyz="0 0 0" rpy="${M_PI/2} 0 0" />
+        <geometry>
+          <cylinder length="${wheel_thickness}" radius="${wheel_radius}"/>
         </geometry>
       </collision>
@@ -96,5 +91,5 @@
         mass="${wheel_mass}" />
     </link>
-    <joint name="${name}_joint" type="fixed">
+    <joint name="${name}_joint" type="continuous">
       <origin xyz="${xyz}" rpy="0 0 0"/>
       <parent link="${parent}"/>
@@ -103,8 +98,8 @@
     </joint>
     <gazebo reference="${name}_link">
-      <mu1>1</mu1>
-      <mu2>1</mu2>
+      <mu1>0.1</mu1>
+      <mu2>0.1</mu2>
       <material>Gazebo/Black</material>
-      <kp>10000000</kp>
+      <kp>1000000</kp>
       <kd>10</kd>
       <selfCollide>false</selfCollide>
@@ -229,5 +224,5 @@
    <origin xyz="${body_length/2} 0 ${body_height/2 - 0.01}"/>
   </joint>
-  <joint name="pico_flexx_axis_to_pico_flexx_holder" type="continuous">
+  <joint name="pico_flexx_angle" type="continuous">
     <parent link="pico_flexx_holder1_link"/>
     <child link="pico_flexx_axis"/>
@@ -324,8 +319,6 @@
       <joint_states_topic_name>joint_states</joint_states_topic_name>
       <left_front_wheel_joint>left_front_wheel_joint</left_front_wheel_joint>
-      <left_middle_wheel_joint>left_middle_wheel_joint</left_middle_wheel_joint>
       <left_rear_wheel_joint>left_rear_wheel_joint</left_rear_wheel_joint>
       <right_front_wheel_joint>right_front_wheel_joint</right_front_wheel_joint>
-      <right_middle_wheel_joint>right_middle_wheel_joint</right_middle_wheel_joint>
       <right_rear_wheel_joint>right_rear_wheel_joint</right_rear_wheel_joint>
       <wheel_separation>${axis_length}</wheel_separation>

Commit message: new wheel mesh

File: ceres_description/urdf/ceres.urdf.xacro (robot description, xacro)
@@ -72,7 +72,8 @@
     <link name="${name}_link">
       <visual>
-        <origin xyz="0 0 0" rpy="${M_PI/2} 0 0" />
-        <geometry>
-          <cylinder length="${wheel_thickness}" radius="${wheel_radius}"/>
+        <origin xyz="0 0 0" rpy="0 0 ${M_PI/2}" />
+        <geometry>
+          <mesh filename="package://ceres_description/meshes/wheel_new.stl"/>
+          <!--cylinder length="${wheel_thickness}" radius="${wheel_radius}"/-->
         </geometry>
         <material name="black" >
@@ -81,7 +82,8 @@
       </visual>
       <collision>
-        <origin xyz="0 0 0" rpy="${M_PI/2} 0 0" />
-        <geometry>
-          <cylinder length="${wheel_thickness}" radius="${wheel_radius}"/>
+        <origin xyz="0 0 0" rpy="0 0 ${M_PI/2}" />
+        <geometry>
+          <mesh filename="package://ceres_description/meshes/wheel_new.stl"/>
+          <!--cylinder length="${wheel_thickness}" radius="${wheel_radius}"/-->
         </geometry>
       </collision>
@@ -98,6 +100,6 @@
     </joint>
     <gazebo reference="${name}_link">
-      <mu1>0.1</mu1>
-      <mu2>0.1</mu2>
+      <mu1>0.8</mu1>
+      <mu2>0.8</mu2>
       <material>Gazebo/Black</material>
       <kp>1000000</kp>

Commit message: new wheel and gazebo controller

File: ceres_description/urdf/ceres.urdf.xacro (robot description, xacro)
@@ -74,6 +74,5 @@
         <origin xyz="0 0 0" rpy="0 0 ${M_PI/2}" />
         <geometry>
-          <mesh filename="package://ceres_description/meshes/wheel_new.stl"/>
-          <!--cylinder length="${wheel_thickness}" radius="${wheel_radius}"/-->
+          <mesh filename="package://ceres_description/meshes/wheel.stl"/>
         </geometry>
         <material name="black" >
@@ -82,8 +81,8 @@
       </visual>
       <collision>
-        <origin xyz="0 0 0" rpy="0 0 ${M_PI/2}" />
-        <geometry>
-          <mesh filename="package://ceres_description/meshes/wheel_new.stl"/>
-          <!--cylinder length="${wheel_thickness}" radius="${wheel_radius}"/-->
+        <origin xyz="0 0 0" rpy="${M_PI/2} 0 0" />
+        <geometry>
+          <!-- mesh filename="package://ceres_description/meshes/wheel.stl"/-->
+          <cylinder length="${wheel_thickness}" radius="${wheel_radius}"/>
         </geometry>
       </collision>
@@ -315,19 +314,17 @@
   <xacro:imu_gazebo link="imu" imu_topic="imu/data" update_rate="100.0" stdev="${imu_stdev}" />
   <gazebo>
-    <plugin name="volksbot_diffdrive" filename="libgazebo_ros_diffdrive_uos.so">
-      <alwaysOn>true</alwaysOn>
-      <cmd_vel_topic_name>cmd_vel</cmd_vel_topic_name>
-      <odom_topic_name>odom</odom_topic_name>
-      <joint_states_topic_name>joint_states</joint_states_topic_name>
-      <left_front_wheel_joint>left_front_wheel_joint</left_front_wheel_joint>
-      <left_rear_wheel_joint>left_rear_wheel_joint</left_rear_wheel_joint>
-      <right_front_wheel_joint>right_front_wheel_joint</right_front_wheel_joint>
-      <right_rear_wheel_joint>right_rear_wheel_joint</right_rear_wheel_joint>
-      <wheel_separation>${axis_length}</wheel_separation>
-      <wheel_diameter>${2*wheel_radius}</wheel_diameter>
-      <turning_adaptation>${turning_adaptation}</turning_adaptation>
-      <torque>4.0</torque>
-      <max_velocity>1.0</max_velocity>
-      <updateRate>40.0</updateRate>
+    <plugin name="skid_steer_drive_controller" filename="libgazebo_ros_skid_steer_drive.so">
+      <updateRate>100.0</updateRate>
+      <robotNamespace>/</robotNamespace>
+      <leftFrontJoint>left_front_wheel_joint</leftFrontJoint>
+      <rightFrontJoint>right_front_wheel_joint</rightFrontJoint>
+      <leftRearJoint>left_rear_wheel_joint</leftRearJoint>
+      <rightRearJoint>right_rear_wheel_joint</rightRearJoint>
+      <wheelSeparation>${axis_length}</wheelSeparation>
+      <wheelDiameter>${2*wheel_radius}</wheelDiameter>
+      <robotBaseFrame>base_link</robotBaseFrame>
+      <torque>20</torque>
+      <topicName>cmd_vel</topicName>
+      <broadcastTF>false</broadcastTF>
     </plugin>
   </gazebo>

Commit message: add recovery behaviors and better diff drive gazebo settings

File: ceres_description/urdf/ceres.urdf.xacro (robot description, xacro)
@@ -16,5 +16,5 @@
   <xacro:property name="axis_front" value="0.14"/>
   <xacro:property name="axis_back" value="-0.14"/>
-  <xacro:property name="wheel_thickness" value="0.085"/>
+  <xacro:property name="wheel_thickness" value="0.025"/>
   <xacro:property name="wheel_body_offset" value="${wheel_thickness/2 + 0.015}"/>
   <xacro:property name="wheel_radius" value="0.135"/>
@@ -23,10 +23,7 @@
   <xacro:property name="axis_left" value="${body_width/2 + wheel_body_offset}"/>
   <xacro:property name="axis_length" value="${body_width + 2 * wheel_body_offset}" />
-  <xacro:property name="turning_adaptation" value="0.95" />
-  <xacro:property name="bearing_width" value="0.05"/>
-  <xacro:property name="bearing_height" value="0.09"/>
-  <xacro:property name="bearing_thickness" value="0.01"/>
-  <xacro:property name="body_mass" value="40.0"/>
-  <xacro:property name="wheel_mass" value="3.0"/>
+  <xacro:property name="turning_adaptation" value="2.95" />
+  <xacro:property name="body_mass" value="25.0"/>
+  <xacro:property name="wheel_mass" value="5.0"/>
   <xacro:property name="imu_width" value="0.036"/>
   <xacro:property name="imu_length" value="0.038"/>
@@ -83,5 +80,4 @@
         <origin xyz="0 0 0" rpy="${M_PI/2} 0 0" />
         <geometry>
-          <!-- mesh filename="package://ceres_description/meshes/wheel.stl"/-->
           <cylinder length="${wheel_thickness}" radius="${wheel_radius}"/>
         </geometry>
@@ -99,9 +95,12 @@
     </joint>
     <gazebo reference="${name}_link">
-      <mu1>0.8</mu1>
-      <mu2>0.8</mu2>
+      <mu1>1.0</mu1>
+      <mu2>1.0</mu2>
       <material>Gazebo/Black</material>
-      <kp>1000000</kp>
-      <kd>10</kd>
+      <kp>100000.0</kp>
+      <kd>10.0</kd>
+      <fdir1>1 0 0</fdir1>
+      <maxVel>1.0</maxVel>
+      <minDepth>0.00</minDepth>
       <selfCollide>false</selfCollide>
     </gazebo>
@@ -314,6 +313,24 @@
   <xacro:imu_gazebo link="imu" imu_topic="imu/data" update_rate="100.0" stdev="${imu_stdev}" />
   <gazebo>
+    <!--plugin name="volksbot_diffdrive" filename="libgazebo_ros_diffdrive_uos.so">
+      <alwaysOn>true</alwaysOn>
+      <cmd_vel_topic_name>cmd_vel</cmd_vel_topic_name>
+      <odom_topic_name>odom</odom_topic_name>
+      <joint_states_topic_name>joint_states</joint_states_topic_name>
+      <left_front_wheel_joint>left_front_wheel_joint</left_front_wheel_joint>
+      <left_middle_wheel_joint>left_middle_wheel_joint</left_middle_wheel_joint>
+      <left_rear_wheel_joint>left_rear_wheel_joint</left_rear_wheel_joint>
+      <right_front_wheel_joint>right_front_wheel_joint</right_front_wheel_joint>
+      <right_middle_wheel_joint>right_middle_wheel_joint</right_middle_wheel_joint>
+      <right_rear_wheel_joint>right_rear_wheel_joint</right_rear_wheel_joint>
+      <wheel_separation>${axis_length}</wheel_separation>
+      <wheel_diameter>${2*wheel_radius}</wheel_diameter>
+      <turning_adaptation>${turning_adaptation}</turning_adaptation>
+      <torque>4.0</torque>
+      <max_velocity>1.4</max_velocity>
+      <updateRate>200.0</updateRate>
+    </plugin-->
     <plugin name="skid_steer_drive_controller" filename="libgazebo_ros_skid_steer_drive.so">
-      <updateRate>100.0</updateRate>
+      <updateRate>200.0</updateRate>
       <robotNamespace>/</robotNamespace>
       <leftFrontJoint>left_front_wheel_joint</leftFrontJoint>

Commit message: use ros control for gazebo sim

File: ceres_description/urdf/ceres.urdf.xacro (robot description, xacro)
@@ -9,4 +9,5 @@
   <xacro:include filename="$(find uos_common_urdf)/urdf/imu.gazebo.urdf.xacro" />
   <xacro:include filename="$(find sick_tim)/urdf/sick_tim.urdf.xacro" />
+  <xacro:include filename="$(find ceres_description)/urdf/wheel.urdf.xacro" />
   <xacro:property name="M_PI" value="3.14159265359"/>
   <xacro:property name="imu_stdev" value="0.00017" />
@@ -65,49 +66,8 @@
     <child link="base_link" />
   </joint>
-  <!--Wheel Macro-->
-  <xacro:macro name="wheel" params="name parent xyz">
+  <xacro:macro name="box_for_joint" params="name r g b color length height width *joint_pose">
     <link name="${name}_link">
       <visual>
-        <origin xyz="0 0 0" rpy="0 0 ${M_PI/2}" />
-        <geometry>
-          <mesh filename="package://ceres_description/meshes/wheel.stl"/>
-        </geometry>
-        <material name="black" >
-          <color rgba="0 0 0 1" />
-        </material>
-      </visual>
-      <collision>
-        <origin xyz="0 0 0" rpy="${M_PI/2} 0 0" />
-        <geometry>
-          <cylinder length="${wheel_thickness}" radius="${wheel_radius}"/>
-        </geometry>
-      </collision>
-      <xacro:cylinder_inertial
-        radius="${wheel_radius}"
-        length="${wheel_thickness}"
-        mass="${wheel_mass}" />
-    </link>
-    <joint name="${name}_joint" type="continuous">
-      <origin xyz="${xyz}" rpy="0 0 0"/>
-      <parent link="${parent}"/>
-      <child link="${name}_link"/>
-      <axis xyz="0 1 0"/>
-    </joint>
-    <gazebo reference="${name}_link">
-      <mu1>1.0</mu1>
-      <mu2>1.0</mu2>
-      <material>Gazebo/Black</material>
-      <kp>100000.0</kp>
-      <kd>10.0</kd>
-      <fdir1>1 0 0</fdir1>
-      <maxVel>1.0</maxVel>
-      <minDepth>0.00</minDepth>
-      <selfCollide>false</selfCollide>
-    </gazebo>
-  </xacro:macro>
-  <xacro:macro name="box_for_joint" params="name o_x o_y o_z r_x r_y r_z r g b color length height width">
-    <link name="${name}_link">
-      <visual>
-        <origin xyz="${o_x} ${o_y} ${o_z}" rpy="${r_x} ${r_y} ${r_z}" />
+        <xacro:insert_block name="joint_pose"/>
         <geometry>
           <box size="${length} ${width} ${height}" />
@@ -119,82 +79,33 @@
     </link>
   </xacro:macro>
-  <xacro:wheel
-    name="left_front_wheel"
-    parent="base_link"
-    xyz="${axis_front} ${axis_left} ${axis_height}" />
-  <xacro:wheel
-    name="left_rear_wheel"
-    parent="base_link"
-    xyz="${axis_back} ${axis_left} ${axis_height}" />
-  <xacro:wheel
-    name="right_front_wheel"
-    parent="base_link"
-    xyz="${axis_front} ${axis_right} ${axis_height}" />
-  <xacro:wheel
-    name="right_rear_wheel"
-    parent="base_link"
-    xyz="${axis_back} ${axis_right} ${axis_height}" />
-  <xacro:sick_tim551
-    name="laser"
-    ros_topic="/scan" />
-  <xacro:box_for_joint
-    name="pico_flexx_holder1"
-    r_x="0"
-    r_y="0"
-    r_z="0"
-    o_x="0"
-    o_y="0"
-    o_z="0"
-    color="silver"
-    r="0.5"
-    g="0.5"
-    b="0.5"
-    length="0.015"
-    width="0.02"
-    height="0.02" />
-  <xacro:box_for_joint
-    name="pico_flexx_holder2"
-    r_x="0"
-    r_y="0"
-    r_z="0"
-    o_x="0"
-    o_y="0"
-    o_z="0"
-    color="silver"
-    r="0.5"
-    g="0.5"
-    b="0.5"
-    length="0.015"
-    width="0.02"
-    height="0.02" />
-  <xacro:box_for_joint
-    name="pico_flexx_model"
-    r_x="0"
-    r_y="0"
-    r_z="0"
-    o_x="0"
-    o_y="0"
-    o_z="0"
-    color="black"
-    r="0"
-    g="0"
-    b="0"
-    length="0.01"
-    width="0.067"
-    height="0.02"/>
- <!--
-  <xacro:box_for_joint
-    name="pico_flexx_bottom_plate"
-    r_x="0"
-    r_y="0"
-    r_z="0"
-    color="silver"
-    r="0.5"
-    g="0.5"
-    b="0.5"
-    length="0.01"
-    width="0.065"
-    height="0.002"/>
-  /-->
+  <xacro:wheel name="left_front_wheel" parent="base_link">
+    <origin xyz="${axis_front} ${axis_left} ${axis_height}" rpy="0 0 0"/>
+  </xacro:wheel>
+  <xacro:wheel name="left_rear_wheel" parent="base_link">
+    <origin xyz="${axis_back} ${axis_left} ${axis_height}" rpy="0 0 0" />
+  </xacro:wheel>
+  <xacro:wheel name="right_front_wheel" parent="base_link">
+    <origin xyz="${axis_front} ${axis_right} ${axis_height}" rpy="0 0 0"/>
+  </xacro:wheel>
+  <xacro:wheel name="right_rear_wheel" parent="base_link">
+    <origin xyz="${axis_back} ${axis_right} ${axis_height}" rpy="0 0 0" />
+  </xacro:wheel>
+  <xacro:sick_tim551 name="laser" ros_topic="/scan" />
+  <xacro:box_for_joint name="pico_flexx_holder1" color="silver" r="0.5" g="0.5" b="0.5"
+                       length="0.015" width="0.02" height="0.02">
+    <origin xyz="0 0 0" rpy="0 0 0" />
+  </xacro:box_for_joint>
+  <xacro:box_for_joint name="pico_flexx_holder2" color="silver" r="0.5" g="0.5" b="0.5"
+                       length="0.015" width="0.02" height="0.02">
+    <origin xyz="0 0 0" rpy="0 0 0" />
+  </xacro:box_for_joint>
+  <xacro:box_for_joint name="pico_flexx_model" color="black" r="0" g="0" b="0"
+                       length="0.01" width="0.067" height="0.02">
+    <origin xyz="0 0 0" rpy="0 0 0" />
+  </xacro:box_for_joint>
+  <!--xacro:box_for_joint name="pico_flexx_bottom_plate" color="silver" r="0.5" g="0.5" b="0.5"
+                      length="0.01" width="0.065" height="0.002">
+    <origin xyz="0 0 0" rpy="0 0 0" />
+  </xacro:box_for_joint-->
   <link name="pico_flexx_optical_frame" type="fixed">
     <visual>
@@ -286,62 +197,20 @@
     <parent link="base_link" />
     <child link="em_body" />
-    <origin
-      xyz=" ${-body_length/2}
-            0.03
-           -0.05
-          " />
+    <origin xyz="${-body_length/2} 0.03 -0.05" />
   </joint>
   <joint name="em_button_to_em_body_joint" type="fixed">
     <parent link="em_body" />
     <child link="em_button" />
-    <origin
-      xyz=" ${-em_button_depth}
-            -0.02
-            0
-          " />
+    <origin xyz=" ${-em_button_depth} -0.02 0" />
   </joint>
   <joint name="imu_to_base_joint" type="fixed">
     <parent link="base_link" />
     <child link="imu" />
-    <origin
-      xyz=" ${imu_offset_x}
-            ${imu_offset_y}
-            ${imu_offset_z}"
-      rpy="${M_PI} 0 ${M_PI/2.0}" />
+    <origin xyz=" ${imu_offset_x} ${imu_offset_y} ${imu_offset_z}" rpy="${M_PI} 0 ${M_PI/2.0}" />
   </joint>
   <!-- inertial measurement unit for gazebo -->
   <xacro:imu_gazebo link="imu" imu_topic="imu/data" update_rate="100.0" stdev="${imu_stdev}" />
   <gazebo>
-    <!--plugin name="volksbot_diffdrive" filename="libgazebo_ros_diffdrive_uos.so">
-      <alwaysOn>true</alwaysOn>
-      <cmd_vel_topic_name>cmd_vel</cmd_vel_topic_name>
-      <odom_topic_name>odom</odom_topic_name>
-      <joint_states_topic_name>joint_states</joint_states_topic_name>
-      <left_front_wheel_joint>left_front_wheel_joint</left_front_wheel_joint>
-      <left_middle_wheel_joint>left_middle_wheel_joint</left_middle_wheel_joint>
-      <left_rear_wheel_joint>left_rear_wheel_joint</left_rear_wheel_joint>
-      <right_front_wheel_joint>right_front_wheel_joint</right_front_wheel_joint>
-      <right_middle_wheel_joint>right_middle_wheel_joint</right_middle_wheel_joint>
-      <right_rear_wheel_joint>right_rear_wheel_joint</right_rear_wheel_joint>
-      <wheel_separation>${axis_length}</wheel_separation>
-      <wheel_diameter>${2*wheel_radius}</wheel_diameter>
-      <turning_adaptation>${turning_adaptation}</turning_adaptation>
-      <torque>4.0</torque>
-      <max_velocity>1.4</max_velocity>
-      <updateRate>200.0</updateRate>
-    </plugin-->
-    <plugin name="skid_steer_drive_controller" filename="libgazebo_ros_skid_steer_drive.so">
-      <updateRate>200.0</updateRate>
-      <robotNamespace>/</robotNamespace>
-      <leftFrontJoint>left_front_wheel_joint</leftFrontJoint>
-      <rightFrontJoint>right_front_wheel_joint</rightFrontJoint>
-      <leftRearJoint>left_rear_wheel_joint</leftRearJoint>
-      <rightRearJoint>right_rear_wheel_joint</rightRearJoint>
-      <wheelSeparation>${axis_length}</wheelSeparation>
-      <wheelDiameter>${2*wheel_radius}</wheelDiameter>
-      <robotBaseFrame>base_link</robotBaseFrame>
-      <torque>20</torque>
-      <topicName>cmd_vel</topicName>
-      <broadcastTF>false</broadcastTF>
+    <plugin name="gazebo_ros_control" filename="libgazebo_ros_control.so">
     </plugin>
   </gazebo>

Commit message: fixed ceres model

File: ceres_description/urdf/ceres.urdf.xacro (robot description, xacro)
@@ -18,5 +18,5 @@
   <xacro:property name="axis_back" value="-0.14"/>
   <xacro:property name="wheel_thickness" value="0.025"/>
-  <xacro:property name="wheel_body_offset" value="${wheel_thickness/2 + 0.015}"/>
+  <xacro:property name="wheel_body_offset" value="${wheel_thickness/2 + 0.035}"/>
   <xacro:property name="wheel_radius" value="0.135"/>
   <xacro:property name="axis_height" value="-0.03"/>
